Commit message: feat: complete NOLO-to-MoveIt simulation baseline

File: vr-xr/src/controller-viewer/public/arm-simulator/models/stararm102_description.urdf (robot description, URDF)
Before this commit: robot stararm102_description, 10 links, 9 joints
Joints:
- joint joint1: limit lower=-2.27 upper=2.27 effort=100 velocity=1 -> lower=-1.9198621772 upper=1.9198621772 effort=100 velocity=1
- joint joint2: limit lower=0 upper=3.14 effort=100 velocity=1 -> lower=0 upper=3.1415926536 effort=100 velocity=1
- joint joint3: limit lower=-3.14 upper=0 effort=100 velocity=1 -> lower=-4.7123889804 upper=0 effort=100 velocity=1
- joint joint4: limit lower=-1.57 upper=2.2 effort=100 velocity=1 -> lower=-1.5707963268 upper=1.5707963268 effort=100 velocity=1
- joint joint5: limit lower=-1.2 upper=1.2 effort=100 velocity=1 -> lower=-1.1344640138 upper=1.1344640138 effort=100 velocity=1
- joint joint6: limit lower=-3.14 upper=3.14 effort=100 velocity=1 -> lower=-2.6179938780 upper=2.6179938780 effort=100 velocity=1
- joint joint7_left: limit lower=0 upper=1.57 effort=5 velocity=3.14 -> lower=0 upper=1.5707963268 effort=5 velocity=3.14
- joint joint7_right: limit lower=-1.57 upper=0 effort=5 velocity=3.14 -> lower=-1.5707963268 upper=0 effort=5 velocity=3.14
